File: Hardware/Star.sch (KiCad schematic (older format))
At the start: 114 parts, among them P1 JTAGICE3, P2 UART, P3 USB_OTG, P4 SPI_FLASH, Q1 BSS806NE, Q10 BSS806NE, Q11 BSS806NE, Q12 BSS806NE, Q13 BSS806NE, Q2 BSS806NE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

Commit message: Finished routing
Connections:
- net GLED_1: now also U3.15 (PA06////SERCOM0.PAD[2]/TCC1.WO[0]); no longer U3.25 (PB12///SERCOM4.PAD[0//TC0.WO[0]/TCC0.WO[6])
- net GLED_2: now also U3.11 (PB08////SERCOM4.PAD[0]/TC0.WO[0]); no longer U3.23 (PB10////SERCOM4.PAD[2]/TC1.WO[0]/TCC0.WO[4])
- net GLED_3: now also U3.17 (PA08///SERCOM0.PAD[0]/SERCOM2.PAD[0]/TCC0.WO[0]/TCC1.WO[2]); no longer U3.19 (PA10///SERCOM0.PAD[2]/SERCOM2.PAD[2]/TCC1.WO[0]/TCC0.WO[2])
- net GLED_4: now also U3.19 (PA10///SERCOM0.PAD[2]/SERCOM2.PAD[2]/TCC1.WO[0]/TCC0.WO[2]); no longer U3.17 (PA08///SERCOM0.PAD[0]/SERCOM2.PAD[0]/TCC0.WO[0]/TCC1.WO[2])
- net GLED_5: now also U3.25 (PB12///SERCOM4.PAD[0//TC0.WO[0]/TCC0.WO[6]); no longer U3.15 (PA06////SERCOM0.PAD[2]/TCC1.WO[0])
- net GLED_6: now also U3.23 (PB10////SERCOM4.PAD[2]/TC1.WO[0]/TCC0.WO[4]); no longer U3.11 (PB08////SERCOM4.PAD[0]/TC0.WO[0])
- net RLED_1: now also U3.16 (PA07////SERCOM0.PAD[3]/TCC1.WO[1]); no longer U3.26 (PB13///SERCOM4.PAD[1]//TC0.WO[1]/TCC0.WO[7])
- net RLED_2: now also U3.12 (PB09////SERCOM4.PAD[1]/TC0.WO[1]); no longer U3.24 (PB11////SERCOM4.PAD[3]/TC1.WO[1]/TCC0.WO[5])
- net RLED_3: now also U3.18 (PA09///SERCOM0.PAD[1]/SERCOM2.PAD[1]/TCC0.WO[1]/TCC1.WO[3]); no longer U3.20 (PA11///SERCOM0.PAD[3]/SERCOM2.PAD[3]/TCC1.WO[1]/TCC0.WO[3])
- net RLED_4: now also U3.20 (PA11///SERCOM0.PAD[3]/SERCOM2.PAD[3]/TCC1.WO[1]/TCC0.WO[3]); no longer U3.18 (PA09///SERCOM0.PAD[1]/SERCOM2.PAD[1]/TCC0.WO[1]/TCC1.WO[3])
- net RLED_5: now also U3.26 (PB13///SERCOM4.PAD[1]//TC0.WO[1]/TCC0.WO[7]); no longer U3.16 (PA07////SERCOM0.PAD[3]/TCC1.WO[1])
- net RLED_6: now also U3.24 (PB11////SERCOM4.PAD[3]/TC1.WO[1]/TCC0.WO[5]); no longer U3.12 (PB09////SERCOM4.PAD[1]/TC0.WO[1])
- net ~PB: now also U3.51 (PA27); no longer U3.13 (PA04/VREFB///SERCOM0.PAD[0]/TCC0.WO[0])
Other:
- moved on the sheet: C18, R28, SW2
Changed lines of the file:
@@
 LIBS:ATSAML21J
 LIBS:Star-cache
-EELAYER 25 0
+EELAYER 26 0
 EELAYER END
 $Descr A3 16535 11693
@@
 Text Notes 9450 7250 0    60   ~ 0
 TCC1.1
+Text GLabel 9825 6750 2    47   Output ~ 0
+GLED_6
+Text GLabel 9825 6650 2    47   Output ~ 0
+RLED_6
+Text GLabel 9825 6550 2    47   Output ~ 0
+GLED_5
+Text GLabel 9825 6450 2    47   Output ~ 0
+RLED_5
+Text GLabel 9825 6950 2    47   Output ~ 0
+GLED_4
+Text GLabel 9825 6850 2    47   Output ~ 0
+RLED_4
+Text GLabel 9825 7150 2    47   Output ~ 0
+GLED_3
+Text GLabel 9825 7050 2    47   Output ~ 0
+RLED_3
 Text GLabel 9825 7750 2    47   Output ~ 0
-GLED_6
+GLED_2
 Text GLabel 9825 7650 2    47   Output ~ 0
-RLED_6
+RLED_2
 Text GLabel 9825 7350 2    47   Output ~ 0
-GLED_5
+GLED_1
 Text GLabel 9825 7250 2    47   Output ~ 0
-RLED_5
-Text GLabel 9825 7150 2    47   Output ~ 0
-GLED_4
-Text GLabel 9825 7050 2    47   Output ~ 0
-RLED_4
-Text GLabel 9825 6950 2    47   Output ~ 0
-GLED_3
-Text GLabel 9825 6850 2    47   Output ~ 0
-RLED_3
-Text GLabel 9825 6750 2    47   Output ~ 0
-GLED_2
-Text GLabel 9825 6650 2    47   Output ~ 0
-RLED_2
-Text GLabel 9825 6550 2    47   Output ~ 0
-GLED_1
-Text GLabel 9825 6450 2    47   Output ~ 0
 RLED_1
 Wire Wire Line
@@
 L SW_PUSH SW2
 U 1 1 584CB794
-P 10750 7350
-F 0 "SW2" V 10796 7296 50  0000 R CNN
-F 1 "PB" V 10705 7296 50  0000 R CNN
-F 2 "Buttons_Switches_SMD:SW_SPST_TL3342" H 10750 7350 50  0001 C CNN
-F 3 "" H 10750 7350 50  0000 C CNN
-	1    10750 7350
+P 14725 5625
+F 0 "SW2" V 14771 5571 50  0000 R CNN
+F 1 "PB" V 14680 5571 50  0000 R CNN
+F 2 "Buttons_Switches_SMD:SW_SPST_TL3342" H 14725 5625 50  0001 C CNN
+F 3 "" H 14725 5625 50  0000 C CNN
+	1    14725 5625
 	0    -1   -1   0
 $EndComp
 Wire Wire Line
-	9375 7550 10425 7550
-Wire Wire Line
-	10750 7050 10750 7025
+	14725 5300 14725 5325
 $Comp
 L C C18
 U 1 1 584D1498
-P 11150 7325
-F 0 "C18" H 11265 7371 50  0000 L CNN
-F 1 "100nF" H 11265 7280 50  0000 L CNN
-F 2 "Capacitors_SMD:C_0603" H 11188 7175 50  0001 C CNN
-F 3 "" H 11150 7325 50  0000 C CNN
-	1    11150 7325
-	1    0    0    -1
-$EndComp
-Wire Wire Line
-	10425 7550 10425 7025
-Wire Wire Line
-	10425 7025 11150 7025
-Wire Wire Line
-	11150 7025 11150 7175
-Connection ~ 10750 7025
-Wire Wire Line
-	10750 7650 10750 7725
-Wire Wire Line
-	10750 7700 11150 7700
-Wire Wire Line
-	11150 7700 11150 7475
+P 15125 5600
+F 0 "C18" H 15240 5646 50  0000 L CNN
+F 1 "100nF" H 15240 5555 50  0000 L CNN
+F 2 "Capacitors_SMD:C_0603" H 15163 5450 50  0001 C CNN
+F 3 "" H 15125 5600 50  0000 C CNN
+	1    15125 5600
+	1    0    0    -1
+$EndComp
+Wire Wire Line
+	14450 5300 15125 5300
+Wire Wire Line
+	15125 5300 15125 5450
+Connection ~ 14725 5300
+Wire Wire Line
+	14725 5925 14725 6000
+Wire Wire Line
+	14725 5975 15125 5975
+Wire Wire Line
+	15125 5975 15125 5750
 $Comp
 L GND #PWR046
 U 1 1 584D2168
-P 10750 7725
-F 0 "#PWR046" H 10750 7475 50  0001 C CNN
-F 1 "GND" H 10755 7552 50  0000 C CNN
-F 2 "" H 10750 7725 50  0000 C CNN
-F 3 "" H 10750 7725 50  0000 C CNN
-	1    10750 7725
-	1    0    0    -1
-$EndComp
-Connection ~ 10750 7700
+P 14725 6000
+F 0 "#PWR046" H 14725 5750 50  0001 C CNN
+F 1 "GND" H 14730 5827 50  0000 C CNN
+F 2 "" H 14725 6000 50  0000 C CNN
+F 3 "" H 14725 6000 50  0000 C CNN
+	1    14725 6000
+	1    0    0    -1
+$EndComp
+Connection ~ 14725 5975
 $Comp
 L R R28
 U 1 1 584D3DBE
-P 10900 6825
-F 0 "R28" H 10950 6875 50  0000 L CNN
-F 1 "10k" H 10950 6775 50  0000 L CNN
-F 2 "Capacitors_SMD:C_0603" V 10830 6825 50  0001 C CNN
-F 3 "" H 10900 6825 50  0000 C CNN
-	1    10900 6825
+P 14875 5100
+F 0 "R28" H 14925 5150 50  0000 L CNN
+F 1 "10k" H 14925 5050 50  0000 L CNN
+F 2 "Capacitors_SMD:C_0603" V 14805 5100 50  0001 C CNN
+F 3 "" H 14875 5100 50  0000 C CNN
+	1    14875 5100
 	-1   0    0    -1
 $EndComp
 Wire Wire Line
-	10900 6975 10900 7025
-Connection ~ 10900 7025
+	14875 5250 14875 5300
+Connection ~ 14875 5300
 $Comp
 L +3V #PWR047
 U 1 1 584D5541
-P 10900 6675
-F 0 "#PWR047" H 10900 6525 50  0001 C CNN
-F 1 "+3V" H 10915 6848 50  0000 C CNN
-F 2 "" H 10900 6675 50  0000 C CNN
-F 3 "" H 10900 6675 50  0000 C CNN
-	1    10900 6675
+P 14875 4950
+F 0 "#PWR047" H 14875 4800 50  0001 C CNN
+F 1 "+3V" H 14890 5123 50  0000 C CNN
+F 2 "" H 14875 4950 50  0000 C CNN
+F 3 "" H 14875 4950 50  0000 C CNN
+	1    14875 4950
 	-1   0    0    -1
 $EndComp
-Text Label 9450 7550 0    47   ~ 0
-~PB
 NoConn ~ 9375 7950
 NoConn ~ 9375 7850
@@
 NoConn ~ 9375 4550
 NoConn ~ 9375 4450
-NoConn ~ 9375 4350
 NoConn ~ 9375 4850
 NoConn ~ 9375 5050
@@
 $EndComp
 $Comp
-L GND #PWR057
+L GND #PWR056
 U 1 1 58545768
 P 8900 9550
-F 0 "#PWR057" H 8900 9300 50  0001 C CNN
+F 0 "#PWR056" H 8900 9300 50  0001 C CNN
 F 1 "GND" H 8905 9377 50  0000 C CNN
 F 2 "" H 8900 9550 50  0000 C CNN
@@
 $EndComp
 $Comp
-L GND #PWR058
+L GND #PWR057
 U 1 1 5847E81F
 P 13800 8000
-F 0 "#PWR058" H 13800 7750 50  0001 C CNN
+F 0 "#PWR057" H 13800 7750 50  0001 C CNN
 F 1 "GND" H 13805 7827 50  0000 C CNN
 F 2 "" H 13800 8000 50  0000 C CNN
@@
 Connection ~ 12000 5050
 $Comp
-L +5V #PWR059
+L +5V #PWR058
 U 1 1 584634AB
 P 11100 5325
-F 0 "#PWR059" H 11100 5175 50  0001 C CNN
+F 0 "#PWR058" H 11100 5175 50  0001 C CNN
 F 1 "+5V" H 11225 5400 50  0000 C CNN
 F 2 "" H 11100 5325 50  0000 C CNN
@@
 	9375 4950 9775 4950
 $Comp
-L +5V #PWR060
+L +5V #PWR059
 U 1 1 5846D809
 P 9925 5025
-F 0 "#PWR060" H 9925 4875 50  0001 C CNN
+F 0 "#PWR059" H 9925 4875 50  0001 C CNN
 F 1 "+5V" H 9925 5175 50  0000 C CNN
 F 2 "" H 9925 5025 50  0000 C CNN
@@
 $EndComp
 $Comp
-L GND #PWR061
+L GND #PWR060
 U 1 1 5847AC2E
 P 9925 5675
-F 0 "#PWR061" H 9925 5425 50  0001 C CNN
+F 0 "#PWR060" H 9925 5425 50  0001 C CNN
 F 1 "GND" H 10075 5600 50  0000 C CNN
 F 2 "" H 9925 5675 50  0000 C CNN
@@
 Wire Wire Line
 	8900 9175 8600 9175
+Text GLabel 9425 4350 2    47   Input ~ 0
+~PB
+Wire Wire Line
+	9375 4350 9425 4350
+Text GLabel 14450 5300 0    47   Output ~ 0
+~PB
+NoConn ~ 9375 7550
 $EndSCHEMATC

Commit message: Finished hardware design
Connections:
- net GND: now also U2.11 (GND), U5.4 (GND), U5.9 (GND)
